File: nrf51822socket/_saved_nrf51822socket.sch (KiCad schematic (older format))
At the start: 14 parts, among them J1 Teste analógico, J2 Esquerdo, J3 Direito, J4 Enable LDO, J5 Input Output, Q1 Q_NMOS_GSD, U1 LN1134

Commit message: Layout do socket para NRF51822 feito
Connections:
- wire segments 71 -> 72
Changed lines of the file:
@@
 L Connector_Generic:Conn_02x09_Odd_Even J2
 U 1 1 5C22DE5C
-P 3750 2650
-F 0 "J2" H 3800 3267 50  0000 C CNN
-F 1 "Esquerdo" H 3800 3176 50  0000 C CNN
-F 2 "Connector_PinSocket_2.00mm:PinSocket_2x09_P2.00mm_Vertical" H 3750 2650 50  0001 C CNN
-F 3 "~" H 3750 2650 50  0001 C CNN
-	1    3750 2650
-	1    0    0    -1
+P 3850 2650
+F 0 "J2" H 3900 3267 50  0000 C CNN
+F 1 "Esquerdo" H 3900 3176 50  0000 C CNN
+F 2 "Connector_PinSocket_2.00mm:PinSocket_2x09_P2.00mm_Vertical" H 3850 2650 50  0001 C CNN
+F 3 "~" H 3850 2650 50  0001 C CNN
+	1    3850 2650
+	-1   0    0    -1
 $EndComp
 $Comp
 L Connector_Generic:Conn_02x09_Odd_Even J3
 U 1 1 5C22DEA6
-P 5450 2650
-F 0 "J3" H 5500 3267 50  0000 C CNN
-F 1 "Direito" H 5500 3176 50  0000 C CNN
-F 2 "Connector_PinSocket_2.00mm:PinSocket_2x09_P2.00mm_Vertical" H 5450 2650 50  0001 C CNN
-F 3 "~" H 5450 2650 50  0001 C CNN
-	1    5450 2650
-	1    0    0    -1
+P 5550 2650
+F 0 "J3" H 5600 3267 50  0000 C CNN
+F 1 "Direito" H 5600 3176 50  0000 C CNN
+F 2 "Connector_PinSocket_2.00mm:PinSocket_2x09_P2.00mm_Vertical" H 5550 2650 50  0001 C CNN
+F 3 "~" H 5550 2650 50  0001 C CNN
+	1    5550 2650
+	-1   0    0    -1
 $EndComp
 $Comp
@@
 SWDIO
 Wire Wire Line
-	5000 2450 5250 2450
+	5000 2450 5150 2450
 Wire Wire Line
 	5950 2450 5750 2450
@@
 	2100 4450 2100 4000
 Connection ~ 2100 4000
+Connection ~ 5150 2450
+Wire Wire Line
+	5150 2450 5250 2450
 $EndSCHEMATC
