File: LowVoltageDCDC/bq25504/bq25504.sch (KiCad schematic (older format))
At the start: 20 parts, among them J1 Conn_01x02, J2 Conn_01x03, J3 Conn_01x02, U1 BQ25504

Commit message: tentativa de conversor tps
Parts:
- U1: symbol Battery_Management:BQ25504 -> bq25504-rescue:BQ25504-Battery_Management
Changed lines of the file:
@@
 	2850 5050 2850 5000
 $Comp
-L Battery_Management:BQ25504 U1
+L bq25504-rescue:BQ25504-Battery_Management U1
 U 1 1 5C10172B
 P 5250 3750
